File: Badge_hw/Badge.sch (KiCad schematic (older format))
At the start: 149 parts

Commit message: *GND circuit, Power Supply modified
Parts:
- removed ANT?: ANT_PCB_MONO, symbol ANT_PCB_MONO
- removed BLN?: BALUN868JOHANSON, Radio:BALUN_JOHANSON868, symbol BALUN868JOHANSON
- removed C? (x2): 0.1uF, symbol C
- removed C? (x17): 10uF, symbol C
- removed C?: 10u, symbol C
- removed C? (x3): 0.1u, symbol C
- removed C?: 1u, symbol C
- removed C? (x2): 18pF, symbol C
- removed C?: 3.9pF, symbol C
- removed C?: DoNotMount, symbol C
- removed C? (x3): 1uF, symbol C
- removed C? (x3): 1nF, symbol C
- removed C?: C, symbol C
- removed D?: CHGLED, symbol LED
- removed DD1: STM32L476Rx, LQFP_TQFP:LQFP64, symbol STM32L476Rx
- removed DD?: STMPE811, QFN_DFN:QFN16_4x4_H, symbol STMPE811
- removed DD?: CC1101, QFN_DFN:QFN20, symbol CC1101
- removed DD?: AXP209, symbol AXP209
- removed DD?: ER-TFT035-6, symbol ER-TFT035-6
- removed L?: BLM15AG102, Inductors:IND_0402, symbol L
- removed L?: 12nH, Inductors:IND_0402, symbol L
- removed L? (x3): 2.2uH, Inductors:IND_0402, symbol L
- removed R? (x2): R, symbol R
- removed R? (x9): 10k, symbol R
- removed R?: 20k, symbol R
- removed R?: 195, symbol R
- removed R?: 240, symbol R
- removed R? (x2): 1, symbol R
- removed R? (x6): 2.2k, symbol R
- removed R?: 200k, symbol R
- removed R?: 0.03, symbol R
- removed SW?: RESET, symbol SW_PUSH_SMALL_H
- removed SW?: PWR_BUT, symbol SW_PUSH_SMALL_H
- removed XTAL? (x2): 27MHz, symbol CRYSTAL_SMD
- added C? (x6): 1u, symbol C
- added C?: 0.22u, symbol C
- added C? (x7): 10u, symbol C
- added C? (x10): 0.1u, symbol C
- added C?: 100p, symbol C
- added C? (x2): 2.2u, symbol C
- added C? (x2): 1n, symbol C
- added C? (x2): 220p, symbol C
- added C? (x2): 10n, symbol C
- added C?: 3.3p, symbol C
- added C?: 18p, symbol C
- added C? (x5): 4.7u, symbol C
- added D? (x2): LED, symbol LED
- added DD?: AXP209, symbol AXP209-RESCUE-Badge
- added L?: BLM15AG102, Inductors:IND_0402, symbol L
- added L? (x3): 4.7u, Inductors:IND_0402, symbol L
- added R?: 470R, symbol R
- added R?: 200k, symbol R
- added R?: 0R03, symbol R
- added R?: 1k, symbol R
- added R?: 2.2k, symbol R
- added R?: 1R, symbol R
- added R? (x2): 4k7, symbol R
- added R?: 51k, symbol R
- added R?: 500R, symbol R
- added R?: 2R2, symbol R
- added R?: 240R, symbol R
- added SW?: SW_PUSH, symbol SW_PUSH
- added XTAL?: 27MHz, CRYSTAL, symbol CRYSTAL_H
- C?: value 22uF -> 22u
- C? (x2): value 0.1uF -> 0.1u
- C?: value 10uF -> 10u
- C?: value C -> 18p
Connections:
- net labels added: +2V5, +3V3_120mA, CHARGING, DB0, DB1, DB2, DB3, DB4, DB5, DB6, DCDC_2, DCDC_3, GNDD, GNDPWR, GNDSignal, LCD_CS, LCD_D/I_SLC, LCD_RD, LCD_RESET, LCD_WR, LCD_X+, LCD_X-, LCD_Y+, LCD_Y-, LDO_1, LDO_3, LX_2, LX_3, MCU_PWR, MCU_RST, PWR_UNST, SCK, SCL, SDA
- net labels removed: +2.2V, 120mA, 2.8V, 3.3V, 60mA, AGND, I2C_SCK, I2C_SDA, IPSOUT, LED_CS, LED_D/I_SLC, LED_RESET, LED_RX, LED_TX, LED_X+, LED_X-, LED_Y+, LED_Y-, MCU_PWR(?), RESET_N, USB_DRV?, VDD, klNFC_VCC, klNFC_Vcc
- wire segments 436 -> 470
- no-connect marks 16 -> 17
Other:
- note added: "100"
- note added: "11"
- note added: "21"
- note added: "22"
- note added: "28"
- note added: "3.3V on \nPWR_ON"
- note added: "50"
- note added: "6"
- note added: "73"
- note added: "75"
- note added: "Debug LED"
- note added: "MCU Power Filter"
- note added: "Pins"
- note added: "VCC from AXP"
- note added: "allow VBUS\nconnect"
- note added: "only DB0..8 pull up"
- moved on the sheet: BLN?, DD?, XTAL?

Commit message: * ground updated
Connections:
- net labels added: DB10, DB11, DB12, DB13, DB14, DB15, DB7, DB8, DB9
- wire segments 470 -> 477

Commit message: *GOST redraw
Parts:
- removed C?: 10u, symbol C
- removed C?: 1n, symbol C
- removed L?: 4.7u, Inductors:IND_0402, symbol L
- removed R? (x7): 10k, symbol R
- added C12: 1n, symbol C-RESCUE-Badge
- added C8: 10u, symbol C-RESCUE-Badge
- added L3: 4.7u, Inductors:IND_0402, symbol L
- added R10, R12, R14, R16, R18, R19, R20: 10k, symbol R-RESCUE-Badge
- C1, C10, C11, C13, C14, C15, C16, C17, C18, C19, C2, C20, C21, C22, C23, C24, C25, C26, C27, C28, C29, C3, C30, C31, C32, C33, C34, C35, C36, C37, C38, C39, C4, C40, C41, C42, C43, C44, C45, C46, C47, C48, C49, C5, C50, C51, C52, C53, C54, C55, C56, C57, C58, C59, C6, C60, C61, C62, C63, C64, C65, C66, C7, C9: renamed from C?; symbol C -> C-RESCUE-Badge
- R1, R11, R13, R15, R17, R2, R21, R22, R23, R24, R25, R26, R27, R28, R29, R3, R30, R31, R32, R33, R34, R35, R36, R37, R38, R39, R4, R40, R5, R6, R7, R8, R9: renamed from R?; symbol R -> R-RESCUE-Badge
- gave numbers to parts that had none: 26
Connections:
- net labels removed: CC_CSK, VCC
- wire segments 477 -> 479
Other:
- note added: "USB connect"
- note removed: "USB connect detection"
- moved on the sheet: DA1A, Q2, SW1

Commit message: update 9.12 - scheme + case updated
Parts:
- removed ANT1: ANT_PCB_MONO, symbol ANT_PCB_MONO
- removed DD4: STM32L476Rx, LQFP_TQFP:LQFP64, symbol STM32L476Rx
- added D4, D5, D6: LED, symbol LED
- added D7: ANT, symbol ANT
- added DD4: STM32L476Vx, LQFP_TQFP:LQFP100, symbol STM32L476Vx
- added R41: 40kR, symbol R-RESCUE-Badge
- added R42, R43, R44, R45: 1kR, symbol R-RESCUE-Badge
- added R?: Fuse0R, symbol R-RESCUE-Badge
- added SA2, SA3: SW_PUSH, symbol SW_PUSH
- C51, C53: value 18pF -> 18p
- D3: symbol DIODE -> DIODE-RESCUE-Badge
- L1, L2, L3, L4, L5, L6, L7: symbol L -> L-RESCUE-Badge
- R2: value 470R -> 1kR
- R31: value 500R -> 1kR
- R35: value 195 -> 195R
- renumbered SW1 to SA1
Connections:
- net labels added: VGND
- net labels removed: GNDD, GNDPWR, MCU_RST
- wire segments 479 -> 516
- no-connect marks 17 -> 44
Other:
- note added: "Battery"
- note added: "I2C PullUp"
- note added: "LCD"
- note added: "POWOK ?"
- note added: "Power supply"
- note added: "RGB LED"
- note removed: "21"
- note removed: "LED"
- moved on the sheet: C1, C10, C11, C12, C13, C15, C16, C17, C18, C19, C2, C21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

Commit message: 9.2 +pcb
Parts:
- removed D4, D5, D6: LED, symbol LED
- added C67: 10u, Capacitors:CAP_0603, symbol C-RESCUE-Badge
- added D4: LED_RGB, LEDs:LED_5050, symbol LED_RGB-RESCUE-Badge
- added TP1: TESTPOINT, PCB:TESTPOINT_1MM, symbol TESTPOINT
- C1, C10, C11, C12, C13, C14, C15, C16, C17, C18, C19, C2, C20, C21, C22, C23, C24, C25, C26, C27, C28, C29, C3, C30, C31, C32, C33, C34, C35, C36, C37, C38, C39, C4, C40, C41, C42, C43, C44, C45, C46, C47, C48, C49, C50, C51, C52, C53, C54, C55, C56, C57, C58, C59, C6, C60, C61, C62, C63, C65, C66, C7, C8, C9: footprint (none) -> Capacitors:CAP_0603
- C5: value 22u -> 10u; footprint (none) -> Capacitors:CAP_0603
- C64: value 3.9pF -> 3.9pF*; footprint (none) -> Capacitors:CAP_0603
- D1, D2: footprint (none) -> LEDs:LED_0603; symbol LED -> LED-RESCUE-Badge
- D3: footprint (none) -> Diodes:SOD80C
- DA1: footprint (none) -> SO_DIL_TSSOP:SO8_208MIL
- DD1: footprint QFN_DFN:QFN16_4x4_H -> LGA:16_4X4_P065
- DD2: footprint (none) -> Connectors:ER-CON50HT-1
- DD3: footprint (none) -> QFN_DFN:QFN48
- L7: value 12nH -> 12nH*
- LIPO_BAT1: footprint (none) -> Connectors:PLS-2
- Q1: footprint (none) -> SOT:SOT23-3
- Q2: value NPN -> BC848; footprint (none) -> SOT:SOT23-3
- R1, R10, R11, R12, R13, R14, R15, R16, R17, R18, R19, R20, R21, R22, R23, R24, R25, R26, R27, R28, R29, R3, R30, R32, R33, R34, R36, R37, R38, R39, R4, R40, R5, R6, R7, R8, R9: footprint (none) -> Resistors:RES_0603
- R2, R31, R42, R43, R44, R45: value 1kR -> 1k; footprint (none) -> Resistors:RES_0603
- R35: value 195R -> 56k; footprint (none) -> Resistors:RES_0603
- R41: value 40kR -> 51k; footprint (none) -> Resistors:RES_0603
- R46: renamed from R?; footprint (none) -> Resistors:RES_0603_FUSE
- SA1, SA2, SA3: footprint (none) -> BtnsSwitches:BTN_6x6_4x4
- XL1: footprint (none) -> Connectors:PLS-6
- XL2: footprint (none) -> Connectors:USBmicro_MOLEX_WM17142
- XL3: footprint (none) -> Connectors:MICROSD_CAP_FIX05A
- XTAL1: footprint (none) -> Quartz:0503x4-4
- XTAL2: footprint CRYSTAL -> Quartz:0503x4-4
Connections:
- net labels added: +3V3
- wire segments 516 -> 520
Other:
- note removed: "Debug LED"
- note removed: "RGB LED"
- moved on the sheet: BLN1, C1, C10, C11, C12, C13, C15, C17, C18, C19, C2, C21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

Commit message: +antenna
Parts:
- D7: footprint (none) -> ANT_868_INV_F:ANTENNA_868_INV_F
Connections:
- wire segments 520 -> 521
Changed lines of the file:
@@
 LIBS:contrib
 LIBS:valves
-LIBS:ns_power
-LIBS:adc_kl
-LIBS:Allwinner
-LIBS:Antennas_kl
-LIBS:Atmel_kl
-LIBS:Audio_kl
-LIBS:Auds
-LIBS:Connectors_kl
-LIBS:dac
-LIBS:display_kl
-LIBS:ESDProtection
-LIBS:Interface_kl
-LIBS:modules
-LIBS:OpAmp_kl
-LIBS:pcb_details
-LIBS:Power_kl
-LIBS:RF ICs
 LIBS:Sensors
-LIBS:SmartCard_kl
-LIBS:st_kl
-LIBS:standard_logic
 LIBS:Switches
-LIBS:Tittar_kl
-LIBS:Transformers
-LIBS:Transistors_kl
 LIBS:Badge-cache1
 LIBS:Badge-cacheGOST
-LIBS:ns_antennas
 LIBS:Badge-cache
 EELAYER 26 0
@@
 F 0 "D7" H 24570 1785 60  0001 C CNN
 F 1 "ANT" H 24365 1815 60  0001 C CNN
-F 2 "" H 24470 1530 60  0001 C CNN
+F 2 "ANT_868_INV_F:ANTENNA_868_INV_F" H 24470 1530 60  0001 C CNN
 F 3 "" H 24470 1530 60  0001 C CNN
 	1    24470 1530
@@
 	1    0    0    -1
 $EndComp
+$Comp
+L GNDSignal #PWR?
+U 1 1 589CC065
+P 24620 1660
+F 0 "#PWR?" H 24670 1710 50  0001 C CNN
+F 1 "GNDSignal" H 20  -190 50  0001 C CNN
+F 2 "" H 20  -90 50  0000 C CNN
+F 3 "" H 20  -90 50  0000 C CNN
+	1    24620 1660
+	1    0    0    -1
+$EndComp
+Wire Wire Line
+	24620 1660 24620 1600
 $EndSCHEMATC

Commit message: * pcb redraw + barometer scheme
Parts:
- added C68: 0.1u, Capacitors:CAP_0603, symbol C-RESCUE-Badge
- added DD6: LPS22HB, QFN_DFN:QFN16_4x4_H, symbol LPS22HB
- added L8: BLM15AG102, Inductors:IND_0402, symbol L-RESCUE-Badge
- C64, C66: footprint Capacitors:CAP_0603 -> Capacitors:CAP_0402
- D7: footprint ANT_868_INV_F:ANTENNA_868_INV_F -> ANT_868_INV_F:ANTENNA_868_INV_F_SHARP
- DD1: footprint LGA:16_4X4_P065 -> QFN_DFN:QFN16_4x4_H
- L1, L3, L4: footprint Inductors:IND_0402 -> Inductors:SDR0805
- L6: footprint Inductors:IND_0402 -> Inductors:IND_SDR0604
- LIPO_BAT1: footprint Connectors:PLS-2 -> Connectors:WB-02(MW-2M)
- R15: footprint Resistors:RES_0603 -> Resistors:RES_1206
- XTAL2: footprint Quartz:0503x4-4 -> Quartz:03225C4
Connections:
- net labels added: PRESSURE_INT
- net labels removed: DCDC_3
- wire segments 521 -> 539
- no-connect marks 44 -> 43
Other:
- note added: "0R03 footprint?"
- note added: "?? Resistor\non I2C_en"
- note added: "???"
- note added: "Barometer"
- moved on the sheet: C44, C46, C49, C50, C52, C55, C58, C63, C65, D3, DA1A, DA1B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

Commit message: * schematic, footprints
Parts:
- C44: value 150pF -> 150p
- C49: value 100pF -> 100p
- C64: value 3.9pF* -> 3.9p*
- DA1: footprint SO_DIL_TSSOP:SO8_208MIL -> SOT:SOT23-8
- DD6: footprint QFN_DFN:QFN16_4x4_H -> LGA:10_2X2
- L1, L3, L4: value 4.7u -> 4.7uH; footprint Inductors:SDR0805 -> Inductors:IND_SDR0604
- L6: footprint Inductors:IND_SDR0604 -> Inductors:IND_1812
- R15: footprint Resistors:RES_1206 -> Resistors:RES_2512
Connections:
- net GNDS: no longer C15.2, C19.2, C3.2, C9.2, DA1.4 (V-)
- new net: C15.2, C19.2, C3.2, C9.2
