File: Badge_hw/Badge.sch (KiCad schematic (older format))
At the start: 147 parts, among them Q1 IRLML9303, Q2 BC848

Commit message: +pcb
Connections:
- net SCK: no longer DD3.2 (SCK)
- net SCL: now also DD3.2 (SCK)
Changed lines of the file:
@@
 SDA
 Text Label 7870 17580 0    60   ~ 0
-SCK
+SCL
 Text Label 7870 17880 0    60   ~ 0
 PWR_IRQ

Commit message: pcb full 1.0
Connections:
- net SCK is gone; now on net SCL: DD4.15 (ADC123-1/LPTIM1_2_IN1/SCL3/LPRX1/PC0)
- net CHARGING: no longer DD4.67 (OTG_SOF/LPTIM2_OUT/MCO/T1C1/CK1/PA8)
- net GNDA: no longer DD2.43 (GND), DD2.48 (GND), DD2.49 (GND), DD2.50 (GND), XL1.3
- net GNDS: now also C15.2, C19.2, C3.2, C9.2, DD2.43 (GND), DD2.48 (GND), DD2.49 (GND), DD2.50 (GND), XL1.3
- no-connect marks 43 -> 44
Changed lines of the file:
@@
 $EndComp
 $Comp
-L GND #PWR01
-U 1 1 58100C58
-P 2700 3840
-F 0 "#PWR01" H 2700 3590 50  0001 C CNN
-F 1 "GND" H 2700 3690 50  0000 C CNN
-F 2 "" H 2700 3840 50  0000 C CNN
-F 3 "" H 2700 3840 50  0000 C CNN
-	1    2700 3840
-	1    0    0    -1
-$EndComp
-$Comp
 L C-RESCUE-Badge C16
 U 1 1 58100C5A
@@
 USB connect
 Text Label 14950 3200 0    60   ~ 0
-SCK
+SCL
 Text Label 15300 2500 0    60   ~ 0
 PWR_IRQ
@@
 $EndComp
 $Comp
-L GND #PWR033
-U 1 1 58188448
-P 29360 3070
-F 0 "#PWR033" H 29360 2820 50  0001 C CNN
-F 1 "GND" H 29360 2920 50  0000 C CNN
-F 2 "" H 29360 3070 50  0000 C CNN
-F 3 "" H 29360 3070 50  0000 C CNN
-	1    29360 3070
-	1    0    0    -1
-$EndComp
-$Comp
 L STMPE811 DD1
 U 1 1 58100C67
@@
 Text Label 14450 1700 0    60   ~ 0
 klNFC_Tx
-Text Label 14500 2300 0    60   ~ 0
-CHARGING
 $Comp
 L AXP209-RESCUE-Badge DD3
@@
 	14350 3400 14950 3400
 Wire Wire Line
-	14500 2300 14350 2300
-Wire Wire Line
 	14350 3600 14960 3600
 Wire Wire Line
@@
 L GNDSignal #PWR0122
 U 1 1 58B0BF46
-P 4150 12700
-F 0 "#PWR0122" H 4200 12750 50  0001 C CNN
-F 1 "GNDSignal" H 4155 12577 50  0000 C CNN
-F 2 "" H -18680 9680 50  0000 C CNN
-F 3 "" H -18680 9680 50  0000 C CNN
-	1    4150 12700
+P 4150 12690
+F 0 "#PWR0122" H 4200 12740 50  0001 C CNN
+F 1 "GNDSignal" H 4155 12567 50  0000 C CNN
+F 2 "" H -18680 9670 50  0000 C CNN
+F 3 "" H -18680 9670 50  0000 C CNN
+	1    4150 12690
 	1    0    0    -1
 $EndComp
@@
 	1    0    0    -1
 $EndComp
+$Comp
+L GNDSignal #PWR?
+U 1 1 58B51BF3
+P 29360 3030
+F 0 "#PWR?" H 29410 3080 50  0001 C CNN
+F 1 "GNDSignal" H 29365 2907 50  0000 C CNN
+F 2 "" H 6530 10  50  0000 C CNN
+F 3 "" H 6530 10  50  0000 C CNN
+	1    29360 3030
+	1    0    0    -1
+$EndComp
+$Comp
+L GNDSignal #PWR?
+U 1 1 58B57A0F
+P 2700 3800
+F 0 "#PWR?" H 2750 3850 50  0001 C CNN
+F 1 "GNDSignal" H 2705 3677 50  0000 C CNN
+F 2 "" H -20130 780 50  0000 C CNN
+F 3 "" H -20130 780 50  0000 C CNN
+	1    2700 3800
+	1    0    0    -1
+$EndComp
+NoConn ~ 14350 2300
 $EndSCHEMATC

Commit message: *pcb 2.0
Connections:
- net +3V3: now also XL1.1; no longer C43.1, C45.1, DD4.21 (VREF+), R41.2, SA3.2
- net MCU_PWR: now also C43.1, C45.1, DD4.21 (VREF+), R41.2, SA3.2; no longer XL1.1
Changed lines of the file:
@@
-$EndComp
-$Comp
-L +3.3V-RESCUE-Badge #PWR065
-U 1 1 58357750
-P 8370 5650
-F 0 "#PWR065" H 8370 5500 50  0001 C CNN
-F 1 "+3.3V" H 8370 5790 50  0000 C CNN
-F 2 "" H 8370 5650 50  0000 C CNN
-F 3 "" H 8370 5650 50  0000 C CNN
-	1    8370 5650
-	0    -1   -1   0
 $EndComp
 $Comp
@@
 $EndComp
 $Comp
-L +3.3V-RESCUE-Badge #PWR072
-U 1 1 584D9AF7
-P 14750 6850
-F 0 "#PWR072" H 14750 6700 50  0001 C CNN
-F 1 "+3.3V" V 14700 7020 50  0000 C CNN
-F 2 "" H 14750 6850 50  0000 C CNN
-F 3 "" H 14750 6850 50  0000 C CNN
-	1    14750 6850
-	0    1    1    0
-$EndComp
-$Comp
 L R-RESCUE-Badge R42
 U 1 1 5850138A
@@
 	1    12900 7310
 	1    0    0    -1
-$EndComp
-$Comp
-L +3.3V-RESCUE-Badge #PWR073
-U 1 1 585331E8
-P 13370 7310
-F 0 "#PWR073" H 13370 7160 50  0001 C CNN
-F 1 "+3.3V" V 13300 7360 50  0000 C CNN
-F 2 "" H 13370 7310 50  0000 C CNN
-F 3 "" H 13370 7310 50  0000 C CNN
-	1    13370 7310
-	0    1    1    0
 $EndComp
 $Comp
@@
 Wire Wire Line
 	5870 16680 6020 16680
-$Comp
-L MCU_PWR #PWR081
-U 1 1 589F5625
-P 29280 2830
-F 0 "#PWR081" H 29280 2680 50  0001 C CNN
-F 1 "MCU_PWR" V 29200 2920 50  0000 C CNN
-F 2 "" H 29280 2830 50  0000 C CNN
-F 3 "" H 29280 2830 50  0000 C CNN
-	1    29280 2830
-	0    1    1    0
-$EndComp
 Wire Wire Line
 	8420 19980 8420 19630
@@
 $EndComp
 NoConn ~ 14350 2300
+$Comp
+L +3.3V-RESCUE-Badge #PWR?
+U 1 1 58BE39AE
+P 29280 2830
+F 0 "#PWR?" H 29280 2680 50  0001 C CNN
+F 1 "+3.3V" V 29230 2880 50  0000 C CNN
+F 2 "" H 29280 2830 50  0000 C CNN
+F 3 "" H 29280 2830 50  0000 C CNN
+	1    29280 2830
+	0    1    1    0
+$EndComp
+$Comp
+L MCU_PWR #PWR?
+U 1 1 58BF0707
+P 8370 5650
+F 0 "#PWR?" H 8370 5500 50  0001 C CNN
+F 1 "MCU_PWR" V 8430 5730 50  0000 C CNN
+F 2 "" H 8370 5650 50  0000 C CNN
+F 3 "" H 8370 5650 50  0000 C CNN
+	1    8370 5650
+	0    -1   -1   0
+$EndComp
+$Comp
+L MCU_PWR #PWR?
+U 1 1 58BF14B5
+P 13370 7310
+F 0 "#PWR?" H 13370 7160 50  0001 C CNN
+F 1 "MCU_PWR" V 13430 7390 50  0000 C CNN
+F 2 "" H 13370 7310 50  0000 C CNN
+F 3 "" H 13370 7310 50  0000 C CNN
+	1    13370 7310
+	0    1    1    0
+$EndComp
+$Comp
+L MCU_PWR #PWR?
+U 1 1 58BF4979
+P 14750 6850
+F 0 "#PWR?" H 14750 6700 50  0001 C CNN
+F 1 "MCU_PWR" V 14810 6930 50  0000 C CNN
+F 2 "" H 14750 6850 50  0000 C CNN
+F 3 "" H 14750 6850 50  0000 C CNN
+	1    14750 6850
+	0    1    1    0
+$EndComp
+$Bitmap
+Pos 31570 20610
+Scale 1,000000
+Data
+89 50 4E 47 0D 0A 1A 0A 00 00 00 0D 49 48 44 52 00 00 01 95 00 00 01 88 08 02 00 00 00 06 71 EA
+29 00 00 00 03 73 42 49 54 08 08 08 DB E1 4F E0 00 00 00 09 70 48 59 73 00 00 12 5C 00 00 12 5C
+01 68 C4 36 89 00 00 07 89 49 44 41 54 78 9C ED DD D1 72 DA 46 18 80 D1 AA E3 F7 7F 65 7A 91 4E
+93 62 01 42 68 91 BF E5 9C 4B 4F A4 9F 71 D8 2F 8B C6 59 2F 97 CB E5 2F 80 A0 BF CF 7E 01 00 3B
+E9 17 50 A5 5F 40 95 7E 01 55 FA 05 54 E9 17 50 A5 5F 40 D5 D7 8E 6B 96 65 59 FD FA 88 1F 25 9B
+75 16 F0 BA 65 FB E2 BC B5 BC BF 7B 7D C1 CF 3A 0B 38 D0 A6 7E 6D 5F E1 7F DA B7 DA 67 9D 05 1C
+EE F1 F3 AF 7D 8B 7C DF 85 B3 CE 02 46 78 D0 AF 17 D7 EA 53 97 CF 3A 0B 18 E4 5E BF 0E 59 A5 1B
+6F 32 EB 2C 60 9C 9B FD 3A 70 7D 3E BC D5 AC B3 80 A1 D6 FB 75 F8 CA BC 73 C3 59 67 01 A3 F9 F9
+55 A0 6A A5 5F 83 F6 14 AB B7 9D 75 16 F0 06 F6 5F 40 95 7E 01 55 D7 FD 1A FA 69 E8 EA E6 B3 CE
+02 DE C3 FE 0B A8 D2 2F A0 4A BF 80 2A FD 02 AA F4 0B A8 D2 2F A0 4A BF 80 AA EB 7E 0D 3D 5C F4
+EA E6 B3 CE 02 DE C3 FE 0B A8 D2 2F A0 6A A5 5F 83 3E 0D AD DE 76 D6 59 C0 1B D8 7F 01 55 EB FD
+3A 7C 4F 71 E7 86 B3 CE 02 46 BB B9 FF 3A 70 65 3E BC D5 AC B3 80 A1 EE 7D 7E 3C 64 7D 6E BC C9
+AC B3 80 71 1E 3C FF 7A 71 95 3E 75 F9 AC B3 80 41 1E 3F BF DF BD 56 77 5C 38 EB 2C 60 84 65 FB
+6A DC 7E CA E8 EB 2B 7C D6 59 C0 81 9E E8 D7 EF 6B 6E 2C F8 11 CB 7B D6 59 C0 EB F6 F4 EB DF 2B
+FF BF DA 87 2E F2 59 67 01 AF F0 F3 AB 40 95 7E 01 55 FA 05 54 E9 17 50 A5 5F 40 95 7E 01 55 FA
+05 54 E9 17 50 A5 5F 40 95 7E 01 55 FA 05 54 E9 17 50 A5 5F 40 95 7E 01 55 FA 05 54 E9 17 50 A5
+5F 40 95 7E 01 55 FA 05 54 E9 17 50 A5 5F 40 95 7E 01 55 FA 05 54 E9 17 50 A5 5F 40 95 7E 01 55
+FA 05 54 E9 17 50 A5 5F 40 95 7E 01 55 FA 05 54 E9 17 50 A5 5F 40 95 7E 01 55 FA 05 54 E9 17 50
+A5 5F 40 95 7E 01 55 FA 05 54 E9 17 50 A5 5F 40 95 7E 01 55 FA 05 54 7D 9D FD 02 3E D4 B2 2C 67
+BF 04 38 CC E5 72 39 65 AE FD D7 09 C4 8B C9 9C F5 96 D6 2F A0 4A BF 80 2A FD 02 AA 3C BF 3F DF
+59 CF 3E E1 15 3F E1 31 AE FD 17 50 A5 5F 40 95 7E 01 55 FA 05 54 E9 17 50 A5 5F 40 95 7E 01 55
+FA 05 54 E9 17 50 A5 5F 40 95 7E 01 55 FA 05 54 E9 17 50 E5 FC 89 AA 9F F0 BF FF 99 49 F1 1C 14
+FB AF 24 F1 E2 70 C5 37 95 7E 01 55 FA 05 54 E9 17 50 E5 F9 FD 0C 8A 4F 5E F9 09 8A CF BC FE 64
+FF 05 54 E9 17 50 A5 5F 40 95 7E 01 55 FA 05 54 E9 17 50 A5 5F 40 95 7E 01 55 FA 05 54 E9 17 50
+A5 5F 40 95 7E 01 55 FA 05 54 39 7F E2 43 D5 0F 1E E0 CA 67 9E 41 62 FF F5 89 C4 6B 3E CB B2 7C
+E0 5F AB 7E C1 3C 3E 2D 61 FA 05 54 E9 17 50 E5 F9 3D 1F FA E8 77 1A 9F F6 99 F1 4F F6 5F 40 95
+7E 01 55 FA 05 54 E9 17 50 A5 5F 40 95 7E 01 55 FA 05 54 E9 17 50 A5 5F 40 95 7E 01 55 FA 05 54
+E9 17 50 A5 5F 40 95 7E 01 55 FA 05 54 E9 17 50 A5 5F 40 95 7E 01 55 FA 05 54 E9 17 50 A5 5F 40
+95 7E 01 55 FA 05 54 E9 17 50 A5 5F 40 95 7E 01 55 FA 05 54 E9 17 50 A5 5F 40 95 7E 01 55 FA 05
+54 E9 17 50 A5 5F 40 95 7E 01 55 FA 05 54 E9 17 50 A5 5F 40 D5 D7 D9 2F 80 8F B3 2C CB EA D7 2F
+97 8B 59 3C 45 BF 78 93 5B CB FB FB 1F 78 7D C1 CF 3A 8B 2B FA C5 70 0F 57 F8 EA 9F DF B7 DA 67
+9D C5 2A CF BF 18 EB D9 45 FE CA 85 B3 CE E2 16 FD 62 A0 17 D7 EA 53 97 CF 3A 8B 3B F4 8B 51 0E
+59 A5 1B 6F 32 EB 2C EE D3 2F 86 38 70 7D 6E 7F 40 3E D9 2C 1E D2 2F 8E 77 F8 CA BC 73 C3 59 67
+B1 85 7E 01 55 FA C5 C1 06 ED 29 56 6F 3B EB 2C 36 D2 2F A0 4A BF 80 2A FD E2 48 43 3F 0D 5D DD
+7C D6 59 6C A7 5F 40 95 7E 01 55 FA 05 54 E9 17 50 A5 5F 40 95 7E 01 55 FA 05 54 E9 17 47 1A 7A
+B8 E8 D5 CD 67 9D C5 76 FA 05 54 E9 17 50 A5 5F 1C 6C D0 A7 A1 D5 DB CE 3A 8B 8D F4 0B A8 D2 2F
+8E 77 F8 9E E2 CE 0D 67 9D C5 16 FA C5 10 07 AE CC 87 B7 9A 75 16 0F E9 17 A3 1C B2 3E 37 DE 64
+D6 59 DC A7 5F 0C F4 E2 2A 7D EA F2 59 67 71 87 7E 31 D6 EE B5 BA E3 C2 59 67 71 CB D7 D9 2F 80
+F9 FD 5A B1 DB 4F 19 7D 65 85 CF 3A 8B 55 FA C5 9B FC B7 7A 6F 2D F8 11 8F C6 27 9B C5 15 9F 1F
+79 B7 EF EB F9 72 B9 8C FB E9 D0 D5 71 F5 59 FC A2 5F 40 95 7E 01 55 FA 05 54 E9 17 50 A5 5F 40
+95 7E 01 55 FA 05 54 E9 17 50 A5 5F 40 95 7E 01 55 FA 05 54 E9 17 50 A5 5F 40 95 7E 01 55 FA 05
+54 E9 17 50 A5 5F 40 95 7E 01 55 FA 05 54 E9 17 50 A5 5F 40 95 7E 01 55 FA 05 54 E9 17 50 A5 5F
+40 95 7E 01 55 FA 05 54 E9 17 50 A5 5F 40 95 7E 01 55 FA 05 54 E9 17 50 A5 5F 40 95 7E 01 55 FA
+05 54 E9 17 50 A5 5F 40 95 7E 01 55 FA 05 54 E9 17 50 A5 5F 40 95 7E 01 55 FA 05 54 E9 17 50 A5
+5F 40 95 7E 01 55 FA 05 54 E9 17 50 A5 5F 40 95 7E 01 55 FA 05 54 E9 17 50 A5 5F 40 95 7E 01 55
+5F 67 BF 00 CE B7 2C CB D9 2F 01 F6 B0 FF 02 AA F4 0B A8 D2 2F A0 4A BF 3E D1 E5 72 39 FB 25 FC
+F6 A3 5E 0C 2D 9E DF 7F 28 D5 60 02 F6 5F 40 95 7E 01 55 FA 05 54 E9 17 50 A5 5F 40 95 7E 01 55
+FA 05 54 E9 17 50 A5 5F 40 95 7E 01 55 FA 05 54 E9 17 50 A5 5F 40 95 7E 01 55 CE CF 99 81 03 EC
+F9 4C F6 5F 40 95 7E 01 55 FA 05 54 E9 57 92 D3 9F 77 F3 AD 9B 89 E7 F7 55 D6 21 D8 7F 01 55 FA
+05 54 E9 17 50 A5 5F 40 95 7E 01 55 FA 05 54 E9 17 50 A5 5F 40 95 7E 01 55 FA 05 54 E9 17 50 A5
+5F 40 95 7E 01 55 FA 05 54 E9 17 50 E5 FC AF F3 F9 ED 1B B0 8F FD 17 50 A5 5F 40 95 7E 9D C0 D1
+CF 70 08 FD 82 51 FC 43 35 9A E7 F7 E7 F0 CE 86 D7 D9 7F 01 55 FA 05 54 E9 17 50 A5 5F 40 95 7E
+01 55 FA 05 54 E9 17 50 A5 5F 40 95 7E 01 55 FA 05 54 E9 17 50 A5 5F 40 95 7E 01 55 FA 05 54 E9
+17 50 A5 5F 40 95 7E 01 55 CE 5F 7D C0 2F 37 83 1F CB FE 0B A8 D2 2F A0 4A BF 80 2A FD BA E6 37
+03 D1 F5 69 EF 5E CF EF 57 7C DA 9B 00 A2 EC BF 80 2A FD 02 AA F4 0B A8 D2 2F A0 4A BF 80 2A FD
+02 AA F4 0B A8 D2 2F A0 4A BF 80 2A FD 02 AA F4 0B A8 D2 2F A0 4A BF 80 2A FD 02 AA 92 E7 E7 38
+93 1E F8 CB FE 0B E8 D2 2F A0 4A BF 80 AA 46 BF 1C E8 0C A3 15 57 59 E6 F9 7D F1 9B 0B 0C D5 D8
+7F 01 7C A7 5F 40 95 7E 01 55 FA 05 54 E9 17 50 A5 5F 40 95 7E 01 55 FA 05 54 E9 17 50 A5 5F 40
+95 7E 01 55 FA 05 54 E9 17 50 A5 5F 40 95 7E 01 55 87 9D FF E5 77 6A 00 6F 66 FF 05 54 E9 17 50
+A5 5F 40 D5 FE 7E 39 90 1E F8 E5 AC 1A 2C 32 04 44 F9 FC 08 54 E9 17 50 A5 5F 40 95 7E 01 55 FA
+05 54 E9 17 50 A5 5F 40 95 7E 01 55 FA 05 54 E9 17 50 A5 5F 40 95 7E 01 55 FA 05 54 E9 17 50 A5
+5F 40 95 7E 01 55 FA 05 54 E9 17 50 A5 5F 40 95 7E 01 55 FA 05 54 E9 17 50 A5 5F 40 95 7E 01 55
+FA 05 54 E9 17 50 A5 5F 40 95 7E 01 55 FA 05 54 FD 03 E5 8A E9 0E 75 88 94 63 00 00 00 00 49 45
+4E 44 AE 42 60 82
+EndData
+$EndBitmap
 $EndSCHEMATC

Commit message: Working FW project
Parts:
- DD3: footprint QFN_DFN:QFN48 -> QFN_DFN:QFN-48_EP_6x6_Pitch0.4mm
