File: Badge_hw/Badge.kicad_pcb (KiCad board)
At the start: 2 copper layers, 114 x 62 mm, 148 parts, among them Q1 IRLML9303, Q2 BC848

Commit message: Working FW project
Routing:
- net GNDS: vias 31 -> 539
- net (no net): vias 508 -> 0
Other:
- rule pad_to_mask_clearance: 0.2 -> 0.1
