File: Badge_hw/Badge.kicad_pcb (KiCad board)
At the start: 2 copper layers, 114 x 62 mm, 148 parts, among them Q1 IRLML9303, Q2 BC848

Commit message: upd
Parts:
- DD3: footprint QFN_DFN:QFN48 -> QFN_DFN:QFN48_EP_6x6_Pitch0.4mm
- moved C39 12.2 mm to (118.1, 73.8)
- moved G*** 1.28 mm to (207.0, 79.7)
- moved DD3 0.36 mm to (130.3, 97.6), turned to 180 degrees
Routing:
- net MCU_PWR: track 178.0 -> 205.2 mm, vias 9 -> 12
- net GNDS: track 495.3 -> 512.6 mm, vias 31 -> 33
- net /ANT2: track 3.45 -> 12.3 mm
- net +3V3: track 297.0 -> 293.0 mm
- net /DCDC_2: track 10.1 -> 13.6 mm
- net Net-(DD4-Pad2): track 13.4 -> 16.4 mm
- net Net-(DD4-Pad3): track 13.2 -> 15.9 mm
- net /PRESSURE_INT: track 56.9 -> 58.3 mm, vias 2 -> 4
- net /DB6: track 31.1 -> 29.8 mm
- net +5V: track 24.0 -> 25.2 mm
- net /DB7: track 30.8 -> 29.7 mm
- net /SCL: track 126.0 -> 127.2 mm
- net /DB5: track 31.9 -> 30.8 mm
- net /PWR_IRQ: track 36.3 -> 37.4 mm
- net /DB10: track 37.9 -> 36.9 mm
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Other:
- outline, holes or cut-outs redrawn
- net class rf added: clearance 0.2, trace_width 0.6, via_dia 0.7, via_drill 0.3
- rule pad_to_mask_clearance: 0.2 -> 0.1
- board text added: "v. 1.05"
