File: Badge/Badge_hw/Badge.kicad_pcb (KiCad board)
At the start: 2 copper layers, 114 x 62 mm, 148 parts, among them Q1 IRLML9303, Q2 BC848

Commit message: badge
Changed lines of the file:
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@@
   (page A4)
   (layers
-    (0 F.Cu signal)
+    (0 F.Cu signal hide)
     (31 B.Cu signal hide)
     (36 B.SilkS user)
-    (37 F.SilkS user)
-    (38 B.Mask user)
-    (39 F.Mask user)
-    (40 Dwgs.User user)
+    (37 F.SilkS user hide)
+    (38 B.Mask user hide)
+    (39 F.Mask user hide)
+    (40 Dwgs.User user hide)
     (44 Edge.Cuts user)
   )
@@
     (pad_to_paste_clearance 0.1)
     (aux_axis_origin 100 112)
-    (visible_elements 7FFFF67F)
+    (visible_elements 7FFFC461)
     (pcbplotparams
-      (layerselection 0x010f0_ffffffff)
+      (layerselection 0x01020_7ffffffe)
       (usegerberextensions true)
-      (excludeedgelayer true)
+      (excludeedgelayer false)
       (linewidth 0.100000)
-      (plotframeref false)
+      (plotframeref true)
       (viasonmask false)
       (mode 1)
@@
       (plotvalue true)
       (plotinvisibletext false)
-      (padsonsilk false)
+      (padsonsilk true)
       (subtractmaskfromsilk false)
-      (outputformat 1)
+      (outputformat 3)
       (mirror false)
       (drillshape 0)
@@
   (module Diodes:SOD80C (layer F.Cu)
     (at 161.4 109.6)
-    (fp_text reference D3 (at 0.2 1.6) (layer F.SilkS)
+    (fp_text reference D3 (at 2.2 1.6) (layer F.SilkS)
       (effects (font (size 0.6 0.6) (thickness 0.15)))
     )
-    (fp_text value PMLL4148 (at -0.12 0.02) (layer F.SilkS)
+    (fp_text value PMLL4148 (at -1.6 1.6) (layer F.SilkS)
       (effects (font (size 0.6 0.6) (thickness 0.15)))
     )
@@
     (descr "Module SOT23")
     (attr smd)
-    (fp_text reference Q2 (at -2.2 -1.6 180) (layer F.SilkS)
+    (fp_text reference Q2 (at -2.4 0 180) (layer F.SilkS)
       (effects (font (size 0.6 0.6) (thickness 0.15)))
     )
-    (fp_text value BC848 (at 0.03 -0.03 180) (layer F.SilkS)
+    (fp_text value BC848 (at 3.2 0 180) (layer F.SilkS)
       (effects (font (size 0.59944 0.59944) (thickness 0.14986)))
     )
